File: RP2040.kicad_sch (KiCad schematic)
At the start: 23 parts, among them J2 Conn_01x02, U26 W25Q128JVS, U27 RP2040, Y1 12.000MHz

Commit message: Bunch more schematic work
Parts:
- added R31, R32, R34: 197, Resistor_SMD:R_0805_2012Metric, symbol Device:R_Small
- added R36, R37, R38: 310, Resistor_SMD:R_0805_2012Metric, symbol Device:R_Small
- added U27: LSF0204PWR, Package_SO:TSSOP-14_4.4x5mm_P0.65mm, symbol Generic-radio-stack:LSF0204PWR
- C19, C20: footprint (none) -> Capacitor_SMD:C_0805_2012Metric
- C21: renamed from C22; footprint (none) -> Capacitor_SMD:C_0805_2012Metric
- C22: renamed from C23; footprint (none) -> Capacitor_SMD:C_0805_2012Metric
- C23: renamed from C24; value C_Small -> 1uF; footprint (none) -> Capacitor_SMD:C_0805_2012Metric
- C24: renamed from C25; footprint (none) -> Capacitor_SMD:C_0805_2012Metric
- C25: renamed from C26; footprint (none) -> Capacitor_SMD:C_0805_2012Metric
- C26: renamed from C27; footprint (none) -> Capacitor_SMD:C_0805_2012Metric
- C27: renamed from C28; footprint (none) -> Capacitor_SMD:C_0805_2012Metric
- C28: renamed from C29; footprint (none) -> Capacitor_SMD:C_0805_2012Metric
- C29: renamed from C30; footprint (none) -> Capacitor_SMD:C_0805_2012Metric
- C30: renamed from C31; footprint (none) -> Capacitor_SMD:C_0805_2012Metric
- C31: renamed from C32; footprint (none) -> Capacitor_SMD:C_0805_2012Metric
- C32: renamed from C21; footprint (none) -> Capacitor_SMD:C_0805_2012Metric
- J2: footprint (none) -> Connector_PinHeader_2.54mm:PinHeader_1x02_P2.54mm_Vertical
- R28: renamed from R26; footprint (none) -> Resistor_SMD:R_0805_2012Metric
- R29: renamed from R27; footprint (none) -> Resistor_SMD:R_0805_2012Metric
- R30: renamed from R28; footprint (none) -> Resistor_SMD:R_0805_2012Metric
- R33: renamed from R24; footprint (none) -> Resistor_SMD:R_0805_2012Metric
- R35: renamed from R25; footprint (none) -> Resistor_SMD:R_0805_2012Metric
- Y1: value 12.000MHz -> ABLS-12.000MHZ-B4-T; footprint (none) -> RP2040_minimal:Crystal_SMD_HC49-US
- renumbered U27 to U26, U26 to U28
Connections:
- net +3V3: now also R31.1, R32.1, R34.1, U27.1 (Vref_A), U27.8 (EN)
- net GND: now also U27.7 (GND)
- net LED_CLOCK: now also R32.2, R37.2, U27.12 (B2), U27.3 (A2)
- net LED_DATA: now also R34.2, R36.2, U27.13 (B1), U27.2 (A1)
- net LED_LOAD: now also R31.2, R38.2, U27.11 (B3), U27.4 (A3)
- net COM1_XFR_LED: now reaches U26.32 (GPIO21)
- net NAV1_XFR_LED: now reaches U26.34 (GPIO22)
- net COM2_XFR_LED: now reaches U26.35 (GPIO23)
- net NAV2_XFR_LED: now reaches U26.36 (GPIO24)
- new net +5V: R36.1, R37.1, R38.1, U27.14 (Vref_B)
- no-connect marks 0 -> 10
Other:
- note added: "Logic level shifting"
- note added: "Place C23 close to pin 45 Place C24 close to pin 44"
- note removed: "Place C24 close to pin 45 Place C25 close to pin 44"
- moved on the sheet: C32, J2, R33, R35, U28

Commit message: Add display footprints and models
Parts:
- C19, C20, C21, C22, C23, C24, C25, C26, C27, C28, C29, C30, C31, C32: footprint Capacitor_SMD:C_0805_2012Metric -> Generic-radio-stack:Perfect_0402
- R28, R29, R30, R31, R32, R33, R34, R36, R37, R38: footprint Resistor_SMD:R_0805_2012Metric -> Generic-radio-stack:Perfect_0402
- R35: value DNF -> 10k; footprint Resistor_SMD:R_0805_2012Metric -> Generic-radio-stack:Perfect_0402
Other:
- note added: "R33 and R35 should be placed close to the flash chip."
Changed lines of the file:
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@@
+    (effects (font (size 1.27 1.27)) (justify left bottom))
+  )
+  (text "R33 and R35 should be placed close\nto the flash chip."
+    (at 193.04 22.86 0)
     (effects (font (size 1.27 1.27)) (justify left bottom))
   )
@@
       (effects (font (size 1.27 1.27)) (justify left))
     )
-    (property "Footprint" "Capacitor_SMD:C_0805_2012Metric" (id 2) (at 144.78 35.56 0)
+    (property "Footprint" "Generic-radio-stack:Perfect_0402" (id 2) (at 144.78 35.56 0)
       (effects (font (size 1.27 1.27)) hide)
     )
@@
       (effects (font (size 1.27 1.27)) (justify left))
     )
-    (property "Footprint" "Capacitor_SMD:C_0805_2012Metric" (id 2) (at 40.64 35.56 0)
+    (property "Footprint" "Generic-radio-stack:Perfect_0402" (id 2) (at 40.64 35.56 0)
       (effects (font (size 1.27 1.27)) hide)
     )
@@
       (effects (font (size 1.27 1.27)) (justify left))
     )
-    (property "Footprint" "Resistor_SMD:R_0805_2012Metric" (id 2) (at 252.73 77.47 0)
+    (property "Footprint" "Generic-radio-stack:Perfect_0402" (id 2) (at 252.73 77.47 0)
       (effects (font (size 1.27 1.27)) hide)
     )
@@
     (property "Reference" "C19" (id 0) (at 21.5963 90.17 90))
     (property "Value" "27p" (id 1) (at 21.5963 92.71 90))
-    (property "Footprint" "Capacitor_SMD:C_0805_2012Metric" (id 2) (at 21.59 96.52 0)
+    (property "Footprint" "Generic-radio-stack:Perfect_0402" (id 2) (at 21.59 96.52 0)
       (effects (font (size 1.27 1.27)) hide)
     )
@@
       (effects (font (size 1.27 1.27)) (justify left))
     )
-    (property "Footprint" "Capacitor_SMD:C_0805_2012Metric" (id 2) (at 167.64 35.56 0)
+    (property "Footprint" "Generic-radio-stack:Perfect_0402" (id 2) (at 167.64 35.56 0)
       (effects (font (size 1.27 1.27)) hide)
     )
@@
       (effects (font (size 1.27 1.27)) (justify left))
     )
-    (property "Footprint" "Resistor_SMD:R_0805_2012Metric" (id 2) (at 210.82 77.47 0)
+    (property "Footprint" "Generic-radio-stack:Perfect_0402" (id 2) (at 210.82 77.47 0)
       (effects (font (size 1.27 1.27)) hide)
     )
@@
     (property "Reference" "R33" (id 0) (at 215.9 36.83 90))
     (property "Value" "1k" (id 1) (at 215.9 39.37 90))
-    (property "Footprint" "Resistor_SMD:R_0805_2012Metric" (id 2) (at 215.9 41.91 0)
+    (property "Footprint" "Generic-radio-stack:Perfect_0402" (id 2) (at 215.9 41.91 0)
       (effects (font (size 1.27 1.27)) hide)
     )
@@
     (property "Reference" "R30" (id 0) (at 125.73 49.53 90))
     (property "Value" "27" (id 1) (at 125.73 52.07 90))
-    (property "Footprint" "Resistor_SMD:R_0805_2012Metric" (id 2) (at 125.73 54.61 0)
+    (property "Footprint" "Generic-radio-stack:Perfect_0402" (id 2) (at 125.73 54.61 0)
       (effects (font (size 1.27 1.27)) hide)
     )
@@
       (effects (font (size 1.27 1.27)) (justify left))
     )
-    (property "Footprint" "Capacitor_SMD:C_0805_2012Metric" (id 2) (at 29.21 35.56 0)
+    (property "Footprint" "Generic-radio-stack:Perfect_0402" (id 2) (at 29.21 35.56 0)
       (effects (font (size 1.27 1.27)) hide)
     )
@@
       (effects (font (size 1.27 1.27)) (justify left))
     )
-    (property "Footprint" "Capacitor_SMD:C_0805_2012Metric" (id 2) (at 133.35 35.56 0)
+    (property "Footprint" "Generic-radio-stack:Perfect_0402" (id 2) (at 133.35 35.56 0)
       (effects (font (size 1.27 1.27)) hide)
     )
@@
       (effects (font (size 1.27 1.27)) (justify left))
     )
-    (property "Footprint" "Resistor_SMD:R_0805_2012Metric" (id 2) (at 267.97 77.47 0)
+    (property "Footprint" "Generic-radio-stack:Perfect_0402" (id 2) (at 267.97 77.47 0)
       (effects (font (size 1.27 1.27)) hide)
     )
@@
       (effects (font (size 1.27 1.27)) (justify left))
     )
-    (property "Footprint" "Capacitor_SMD:C_0805_2012Metric" (id 2) (at 52.07 35.56 0)
+    (property "Footprint" "Generic-radio-stack:Perfect_0402" (id 2) (at 52.07 35.56 0)
       (effects (font (size 1.27 1.27)) hide)
     )
@@
       (effects (font (size 1.27 1.27)) (justify left))
     )
-    (property "Footprint" "Capacitor_SMD:C_0805_2012Metric" (id 2) (at 121.92 35.56 0)
+    (property "Footprint" "Generic-radio-stack:Perfect_0402" (id 2) (at 121.92 35.56 0)
       (effects (font (size 1.27 1.27)) hide)
     )
@@
       (effects (font (size 1.27 1.27)) (justify left))
     )
-    (property "Footprint" "Capacitor_SMD:C_0805_2012Metric" (id 2) (at 247.65 26.67 0)
+    (property "Footprint" "Generic-radio-stack:Perfect_0402" (id 2) (at 247.65 26.67 0)
       (effects (font (size 1.27 1.27)) hide)
     )
@@
       (effects (font (size 1.27 1.27)) (justify left))
     )
-    (property "Footprint" "Capacitor_SMD:C_0805_2012Metric" (id 2) (at 156.21 35.56 0)
+    (property "Footprint" "Generic-radio-stack:Perfect_0402" (id 2) (at 156.21 35.56 0)
       (effects (font (size 1.27 1.27)) hide)
     )
@@
       (effects (font (size 1.27 1.27)) (justify left))
     )
-    (property "Footprint" "Capacitor_SMD:C_0805_2012Metric" (id 2) (at 77.47 26.67 0)
+    (property "Footprint" "Generic-radio-stack:Perfect_0402" (id 2) (at 77.47 26.67 0)
       (effects (font (size 1.27 1.27)) hide)
     )
@@
       (effects (font (size 1.27 1.27)) (justify left))
     )
-    (property "Footprint" "Capacitor_SMD:C_0805_2012Metric" (id 2) (at 179.07 35.56 0)
+    (property "Footprint" "Generic-radio-stack:Perfect_0402" (id 2) (at 179.07 35.56 0)
       (effects (font (size 1.27 1.27)) hide)
     )
@@
     (property "Reference" "C20" (id 0) (at 21.59 110.49 90))
     (property "Value" "27p" (id 1) (at 21.59 107.95 90))
-    (property "Footprint" "Capacitor_SMD:C_0805_2012Metric" (id 2) (at 21.59 104.14 0)
+    (property "Footprint" "Generic-radio-stack:Perfect_0402" (id 2) (at 21.59 104.14 0)
       (effects (font (size 1.27 1.27)) hide)
     )
@@
       (effects (font (size 1.27 1.27)) (justify left))
     )
-    (property "Footprint" "Capacitor_SMD:C_0805_2012Metric" (id 2) (at 110.49 35.56 0)
+    (property "Footprint" "Generic-radio-stack:Perfect_0402" (id 2) (at 110.49 35.56 0)
       (effects (font (size 1.27 1.27)) hide)
     )
@@
     (property "Reference" "R29" (id 0) (at 125.73 41.91 90))
     (property "Value" "27" (id 1) (at 125.73 44.45 90))
-    (property "Footprint" "Resistor_SMD:R_0805_2012Metric" (id 2) (at 125.73 46.99 0)
+    (property "Footprint" "Generic-radio-stack:Perfect_0402" (id 2) (at 125.73 46.99 0)
       (effects (font (size 1.27 1.27)) hide)
     )
@@
     (property "Reference" "R28" (id 0) (at 43.18 99.06 90))
     (property "Value" "1k" (id 1) (at 43.18 101.6 90))
-    (property "Footprint" "Resistor_SMD:R_0805_2012Metric" (id 2) (at 43.18 104.14 0)
+    (property "Footprint" "Generic-radio-stack:Perfect_0402" (id 2) (at 43.18 104.14 0)
       (effects (font (size 1.27 1.27)) hide)
     )
@@
       (effects (font (size 1.27 1.27)) (justify left))
     )
-    (property "Footprint" "Resistor_SMD:R_0805_2012Metric" (id 2) (at 218.44 77.47 0)
+    (property "Footprint" "Generic-radio-stack:Perfect_0402" (id 2) (at 218.44 77.47 0)
       (effects (font (size 1.27 1.27)) hide)
     )
@@
       (effects (font (size 1.27 1.27)) (justify left))
     )
-    (property "Footprint" "Resistor_SMD:R_0805_2012Metric" (id 2) (at 260.35 77.47 0)
+    (property "Footprint" "Generic-radio-stack:Perfect_0402" (id 2) (at 260.35 77.47 0)
       (effects (font (size 1.27 1.27)) hide)
     )
@@
       (effects (font (size 1.27 1.27)) (justify left))
     )
-    (property "Value" "DNF" (id 1) (at 233.68 27.9399 0)
-      (effects (font (size 1.27 1.27)) (justify left))
-    )
-    (property "Footprint" "Resistor_SMD:R_0805_2012Metric" (id 2) (at 231.14 26.67 0)
+    (property "Value" "10k" (id 1) (at 233.68 27.9399 0)
+      (effects (font (size 1.27 1.27)) (justify left))
+    )
+    (property "Footprint" "Generic-radio-stack:Perfect_0402" (id 2) (at 231.14 26.67 0)
       (effects (font (size 1.27 1.27)) hide)
     )
@@
       (effects (font (size 1.27 1.27)) (justify left))
     )
-    (property "Footprint" "Resistor_SMD:R_0805_2012Metric" (id 2) (at 203.2 77.47 0)
-      (effects (font (size 1.27 1.27)) hide)
-    )
+    (property "Footprint" "Generic-radio-stack:Perfect_0402" (id 2) (at 203.2 77.47 0)
+      (effects (font (size 1.27 1.27)) hide)
+    )

Commit message: Custom component for six digit display
Parts:
- renumbered U26 to U22, U27 to U23, U28 to U24
Changed lines of the file:
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@@
   (symbol (lib_id "Memory_Flash:W25Q128JVS") (at 243.84 44.45 0) (unit 1)
     (in_bom yes) (on_board yes)
-    (property "Reference" "U28" (id 0) (at 233.68 53.34 0)
+    (property "Reference" "U24" (id 0) (at 233.68 53.34 0)
       (effects (font (size 1.27 1.27)) (justify left))
     )
@@
   (symbol (lib_id "Generic-radio-stack:LSF0204PWR") (at 237.49 86.36 0) (unit 1)
     (in_bom yes) (on_board yes)
-    (property "Reference" "U27" (id 0) (at 237.49 71.12 0))
+    (property "Reference" "U23" (id 0) (at 237.49 71.12 0))
     (property "Value" "LSF0204PWR" (id 1) (at 237.49 73.66 0))
     (property "Footprint" "Package_SO:TSSOP-14_4.4x5mm_P0.65mm" (id 2) (at 237.49 102.87 0)
@@
   (symbol (lib_id "MCU_RaspberryPi_RP2040:RP2040") (at 86.36 95.25 0) (unit 1)
     (in_bom yes) (on_board yes) (fields_autoplaced)
-    (property "Reference" "U26" (id 0) (at 88.3794 146.05 0)
-      (effects (font (size 1.27 1.27)) (justify left))
-    )
+    (property "Reference" "U22" (id 0) (at 88.3794 146.05 0)
+      (effects (font (size 1.27 1.27)) (justify left))
+    )

Commit message: More footprint updates
Parts:
- renumbered U22 to U18, U23 to U19, U24 to U20
Changed lines of the file:
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@@
   (symbol (lib_id "Memory_Flash:W25Q128JVS") (at 243.84 44.45 0) (unit 1)
     (in_bom yes) (on_board yes)
-    (property "Reference" "U24" (id 0) (at 233.68 53.34 0)
+    (property "Reference" "U20" (id 0) (at 233.68 53.34 0)
       (effects (font (size 1.27 1.27)) (justify left))
     )
@@
   (symbol (lib_id "Generic-radio-stack:LSF0204PWR") (at 237.49 86.36 0) (unit 1)
     (in_bom yes) (on_board yes)
-    (property "Reference" "U23" (id 0) (at 237.49 71.12 0))
+    (property "Reference" "U19" (id 0) (at 237.49 71.12 0))
     (property "Value" "LSF0204PWR" (id 1) (at 237.49 73.66 0))
     (property "Footprint" "Package_SO:TSSOP-14_4.4x5mm_P0.65mm" (id 2) (at 237.49 102.87 0)
@@
   (symbol (lib_id "MCU_RaspberryPi_RP2040:RP2040") (at 86.36 95.25 0) (unit 1)
     (in_bom yes) (on_board yes) (fields_autoplaced)
-    (property "Reference" "U22" (id 0) (at 88.3794 146.05 0)
-      (effects (font (size 1.27 1.27)) (justify left))
-    )
+    (property "Reference" "U18" (id 0) (at 88.3794 146.05 0)
+      (effects (font (size 1.27 1.27)) (justify left))
+    )

Commit message: initial routing of RP2040
Connections:
- net +3V3: now also U18.44 (VREG_IN)
- net GND: no longer U18.44 (VREG_IN)
- net XIN: now reaches C19.2, U18.20 (XIN)
- net XIN: now also Y1.1; no longer Y1.2
- net D-: now reaches R30.1, U18.46 (USB_DM)
- net at C20.2, R28.1: now also Y1.2; no longer Y1.1
- net D+: now reaches R29.1, U18.47 (USB_DP)
- net XOUT: now reaches R28.2, U18.21 (XOUT)
Other:
- note added: "Pins 48 and 49 share C25"
- moved on the sheet: C24, Y1
Changed lines of the file:
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@@
   (junction (at 31.75 104.14) (diameter 0) (color 0 0 0 0)
   )
+  (junction (at 77.47 27.94) (diameter 0) (color 0 0 0 0)
+  )
   (junction (at 121.92 38.1) (diameter 0) (color 0 0 0 0)
   )
@@
   )
   (junction (at 90.17 44.45) (diameter 0) (color 0 0 0 0)
-  )
-  (junction (at 77.47 29.21) (diameter 0) (color 0 0 0 0)
   )
   (junction (at 144.78 33.02) (diameter 0) (color 0 0 0 0)
@@
     (stroke (width 0) (type default) (color 0 0 0 0))
   )
-  (wire (pts (xy 80.01 29.21) (xy 80.01 31.75))
+  (wire (pts (xy 80.01 33.02) (xy 80.01 35.56))
     (stroke (width 0) (type default) (color 0 0 0 0))
   )
@@
     (stroke (width 0) (type default) (color 0 0 0 0))
   )
-  (wire (pts (xy 77.47 29.21) (xy 80.01 29.21))
-    (stroke (width 0) (type default) (color 0 0 0 0))
-  )
   (wire (pts (xy 99.06 44.45) (xy 102.87 44.45))
     (stroke (width 0) (type default) (color 0 0 0 0))
@@
     (stroke (width 0) (type default) (color 0 0 0 0))
   )
+  (wire (pts (xy 77.47 27.94) (xy 80.01 27.94))
+    (stroke (width 0) (type default) (color 0 0 0 0))
+  )
   (wire (pts (xy 29.21 33.02) (xy 40.64 33.02))
     (stroke (width 0) (type default) (color 0 0 0 0))
@@
     (stroke (width 0) (type default) (color 0 0 0 0))
   )
+  (wire (pts (xy 77.47 27.94) (xy 77.47 44.45))
+    (stroke (width 0) (type default) (color 0 0 0 0))
+  )
   (wire (pts (xy 226.06 87.63) (xy 203.2 87.63))
     (stroke (width 0) (type default) (color 0 0 0 0))
@@
     (stroke (width 0) (type default) (color 0 0 0 0))
   )
-  (wire (pts (xy 77.47 29.21) (xy 77.47 44.45))
+  (wire (pts (xy 77.47 24.13) (xy 77.47 27.94))
     (stroke (width 0) (type default) (color 0 0 0 0))
   )
@@
   (wire (pts (xy 24.13 96.52) (xy 31.75 96.52))
     (stroke (width 0) (type default) (color 0 0 0 0))
+  )
+  (text "Pins 48 and 49 share C25" (at 110.49 31.75 0)
+    (effects (font (size 1.27 1.27)) (justify left bottom))
   )
   (text "Flash" (at 190.5 15.24 0)
@@
     (effects (font (size 1.27 1.27)) (justify right bottom))
   )
+  (label "XOUT" (at 54.61 102.87 180)
+    (effects (font (size 1.27 1.27)) (justify right bottom))
+  )
   (label "LED_DATA" (at 130.81 72.39 180)
     (effects (font (size 1.27 1.27)) (justify right bottom))
@@
     (effects (font (size 1.27 1.27)) (justify right bottom))
   )
+  (label "D-" (at 118.11 54.61 0)
+    (effects (font (size 1.27 1.27)) (justify left bottom))
+  )
+  (label "D+" (at 118.11 52.07 0)
+    (effects (font (size 1.27 1.27)) (justify left bottom))
+  )
   (label "QSPI_SD0" (at 270.51 39.37 180)
+    (effects (font (size 1.27 1.27)) (justify right bottom))
+  )
+  (label "XIN" (at 54.61 97.79 180)
     (effects (font (size 1.27 1.27)) (justify right bottom))
   )
@@
     (pin "1")
   )
-  (symbol (lib_id "power:GND") (at 80.01 31.75 0) (unit 1)
-    (in_bom yes) (on_board yes) (fields_autoplaced)
-    (property "Reference" "#PWR052" (id 0) (at 80.01 38.1 0)
-      (effects (font (size 1.27 1.27)) hide)
-    )
-    (property "Value" "GND" (id 1) (at 80.01 36.83 0))
-    (property "Footprint" "" (id 2) (at 80.01 31.75 0)
-      (effects (font (size 1.27 1.27)) hide)
-    )
-    (property "Datasheet" "" (id 3) (at 80.01 31.75 0)
+  (symbol (lib_id "power:GND") (at 80.01 35.56 0) (unit 1)
+    (in_bom yes) (on_board yes) (fields_autoplaced)
+    (property "Reference" "#PWR052" (id 0) (at 80.01 41.91 0)
+      (effects (font (size 1.27 1.27)) hide)
+    )
+    (property "Value" "GND" (id 1) (at 80.01 40.64 0))
+    (property "Footprint" "" (id 2) (at 80.01 35.56 0)
+      (effects (font (size 1.27 1.27)) hide)
+    )
+    (property "Datasheet" "" (id 3) (at 80.01 35.56 0)
       (effects (font (size 1.27 1.27)) hide)
     )
@@
     (pin "1")
   )
-  (symbol (lib_id "Device:C_Small") (at 77.47 26.67 0) (unit 1)
-    (in_bom yes) (on_board yes) (fields_autoplaced)
-    (property "Reference" "C24" (id 0) (at 80.01 25.4062 0)
-      (effects (font (size 1.27 1.27)) (justify left))
-    )
-    (property "Value" "1uF" (id 1) (at 80.01 27.9462 0)
-      (effects (font (size 1.27 1.27)) (justify left))
-    )
-    (property "Footprint" "Generic-radio-stack:Perfect_0402" (id 2) (at 77.47 26.67 0)
-      (effects (font (size 1.27 1.27)) hide)
-    )
-    (property "Datasheet" "~" (id 3) (at 77.47 26.67 0)
+  (symbol (lib_id "Device:C_Small") (at 80.01 30.48 0) (unit 1)
+    (in_bom yes) (on_board yes) (fields_autoplaced)
+    (property "Reference" "C24" (id 0) (at 82.55 29.2162 0)
+      (effects (font (size 1.27 1.27)) (justify left))
+    )
+    (property "Value" "1uF" (id 1) (at 82.55 31.7562 0)
+      (effects (font (size 1.27 1.27)) (justify left))
+    )
+    (property "Footprint" "Generic-radio-stack:Perfect_0402" (id 2) (at 80.01 30.48 0)
+      (effects (font (size 1.27 1.27)) hide)
+    )
+    (property "Datasheet" "~" (id 3) (at 80.01 30.48 0)
       (effects (font (size 1.27 1.27)) hide)
     )
@@
     (pin "9")
   )
-  (symbol (lib_id "Device:Crystal") (at 31.75 100.33 90) (unit 1)
+  (symbol (lib_id "Device:Crystal") (at 31.75 100.33 270) (unit 1)
     (in_bom yes) (on_board yes)
-    (property "Reference" "Y1" (id 0) (at 30.48 93.98 90)
+    (property "Reference" "Y1" (id 0) (at 33.02 106.68 90)
       (effects (font (size 1.27 1.27)) (justify right))
     )
-    (property "Value" "ABLS-12.000MHZ-B4-T" (id 1) (at 26.67 106.68 90)
+    (property "Value" "ABLS-12.000MHZ-B4-T" (id 1) (at 36.83 93.98 90)
       (effects (font (size 1.27 1.27)) (justify right))
     )
